File: pygameboy.sch (KiCad schematic (older format))
At the start: 32 parts, among them J1 Conn_01x01, J2 Conn_01x01, J3 Conn_ARM_JTAG_SWD_10, J4 USB_B_Micro, Q1 BSS138, U1 CARTRIDGE, U2 SAMD51J, U3 74LS244, U4 74LS244, U5 74x4245, U6 74LS244, U7 AP2204K-3.3

Commit message: v2 with added caps. reworked CCL signals and lotsa test points
Parts:
- added C14: 10uF, Capacitors_SMD:C_0603_HandSoldering, symbol device:C_Small
- added C15: 1uF, Capacitors_SMD:C_0603_HandSoldering, symbol device:C_Small
- added TP1, TP10, TP11, TP12, TP13, TP14, TP15, TP16, TP17, TP18, TP19, TP2, TP20, TP21, TP22, TP23, TP24, TP25, TP26, TP27, TP28, TP29, TP3, TP30, TP31, TP32, TP4, TP5, TP6, TP7, TP8, TP9: Test_Point, gameboy:Test Point, symbol Connector:Test_Point
- added TP33: Test_Point, keystone:5015-SMT-TestPoint, symbol Connector:Test_Point
- added TP34: DATA_OE, keystone:5015-SMT-TestPoint, symbol Connector:Test_Point
- added TP35: GB_RESET, keystone:5015-SMT-TestPoint, symbol Connector:Test_Point
- added TP36: SAMD_RESET, keystone:5015-SMT-TestPoint, symbol Connector:Test_Point
- added TP37: gnd, keystone:5015-SMT-TestPoint, symbol Connector:Test_Point
- added TP38: 3.3v, keystone:5015-SMT-TestPoint, symbol Connector:Test_Point
- added TP39: batt, keystone:5015-SMT-TestPoint, symbol Connector:Test_Point
- added TP40: clk, keystone:5015-SMT-TestPoint, symbol Connector:Test_Point
- added TP41: rd, keystone:5015-SMT-TestPoint, symbol Connector:Test_Point
- added TP42: wr, keystone:5015-SMT-TestPoint, symbol Connector:Test_Point
- added TP43: a15, keystone:5015-SMT-TestPoint, symbol Connector:Test_Point
- added TP44: PB17, keystone:5015-SMT-TestPoint, symbol Connector:Test_Point
- added TP45: cs, keystone:5015-SMT-TestPoint, symbol Connector:Test_Point
Connections:
- net labels added: SWO
- wire segments 53 -> 55
- no-connect marks 10 -> 9

Commit message: v3
Parts:
- added C16, C17: C_Small, Capacitor_SMD:C_0603_1608Metric_Pad1.05x0.95mm_HandSolder, symbol Device:C_Small
- added D4: 1N4148W, Diode_SMD:D_SOD-123, symbol Diode:1N4148W
- added J5: MIDI IN, cui-audio:CUI_SJ-3523-SMT-TR, symbol Connector:AudioJack3_Ground
- added J6: MIDI OUT, cui-audio:CUI_SJ-3523-SMT-TR, symbol Connector:AudioJack3_Ground
- added R5, R6, R7: R_Small, Resistor_SMD:R_0603_1608Metric_Pad1.05x0.95mm_HandSolder, symbol Device:R_Small
- added R8: 10k, Resistor_SMD:R_0603_1608Metric_Pad1.05x0.95mm_HandSolder, symbol Device:R_Small
- added TP46: data0, keystone:5015-SMT-TestPoint, symbol pygameboy-rescue:Test_Point-Connector
- added TP47: D0, keystone:5015-SMT-TestPoint, symbol pygameboy-rescue:Test_Point-Connector
- added U8: 6N137S, Package_DIP:SMDIP-8_W9.53mm, symbol Isolator:6N136S
- C1, C11, C12, C13, C14, C15, C2, C3, C4, C5, C6, C7, C9: symbol device:C_Small -> pygameboy-rescue:C_Small-device
- C10, C8: symbol device:C_Small -> Device:C_Small
- D1, D2: symbol device:D_Schottky -> pygameboy-rescue:D_Schottky-device
- D3: symbol device:LED -> pygameboy-rescue:LED-device
- J1, J2: symbol Connector:Conn_01x01 -> pygameboy-rescue:Conn_01x01-Connector
- Q1: symbol Transistor:BSS138 -> pygameboy-rescue:BSS138-Transistor
- R1, R2, R3, R4: symbol device:R_Small -> pygameboy-rescue:R_Small-device
- TP1, TP10, TP11, TP12, TP13, TP14, TP15, TP16, TP17, TP18, TP19, TP2, TP20, TP21, TP22, TP23, TP24, TP25, TP26, TP27, TP28, TP29, TP3, TP30, TP31, TP32, TP33, TP34, TP35, TP36, TP37, TP38, TP39, TP4, TP40, TP41, TP42, TP43, TP44, TP45, TP5, TP6, TP7, TP8, TP9: symbol Connector:Test_Point -> pygameboy-rescue:Test_Point-Connector
- U3, U4, U6: symbol Logic_74xx:74LS244 -> pygameboy-rescue:74LS244-Logic_74xx
- U7: symbol regul:AP2204K-3.3 -> pygameboy-rescue:AP2204K-3.3-regul
Connections:
- net labels added: MIDI_IN, MIDI_OUT, SHIELD
- wire segments 55 -> 75
- no-connect marks 9 -> 10
Other:
- moved on the sheet: J4

Commit message: Fixup MIDI and switch to Adafruit parts
Parts:
- removed J5: MIDI IN, cui-audio:CUI_SJ-3523-SMT-TR, symbol Connector:AudioJack3_Ground
- removed J6: MIDI OUT, cui-audio:CUI_SJ-3523-SMT-TR, symbol Connector:AudioJack3_Ground
- removed R8: 10k, Resistor_SMD:R_0603_1608Metric_Pad1.05x0.95mm_HandSolder, symbol Device:R_Small
- removed U8: 6N137S, Package_DIP:SMDIP-8_W9.53mm, symbol Isolator:6N136S
- added J5: MIDI IN, adafruit:4UCONN_19269_TRS, symbol Connector:AudioJack3_SwitchTR
- added J6: MIDI OUT, adafruit:4UCONN_19269_TRS, symbol Connector:AudioJack3_SwitchTR
- added SW1: SW_Push, Button_Switch_SMD:SW_SPST_KMR2, symbol Switch:SW_Push
- added U8: H11L1, Package_DIP:SMDIP-6_W7.62mm, symbol Isolator:H11L1
- C1, C10, C11, C12, C13, C14, C15, C2, C3, C4, C5, C6, C7, C8, C9: footprint Capacitors_SMD:C_0603_HandSoldering -> Capacitor_SMD:C_0603_1608Metric_Pad1.05x0.95mm_HandSolder
- D1, D2: footprint Diodes_SMD:D_SOD-123 -> Diode_SMD:D_SOD-123
- D3: footprint LEDs:LED_0603_HandSoldering -> LED_SMD:LED_0603_1608Metric_Pad1.05x0.95mm_HandSolder
- J4: footprint fci:Mini-USB-B-OshPark -> adafruit:4UCONN_20329_V2_USB
- R1, R2, R3, R4: footprint Resistors_SMD:R_0603_HandSoldering -> Resistor_SMD:R_0603_1608Metric_Pad1.05x0.95mm_HandSolder
- R5: value R_Small -> 220
- R6, R7: value R_Small -> 51
- U2: footprint Housings_QFP:LQFP-64_10x10mm_Pitch0.5mm -> Package_QFP:LQFP-64_10x10mm_P0.5mm
- U3, U4, U6: footprint Housings_SSOP:TSSOP-20_4.4x6.5mm_Pitch0.65mm -> Package_SO:TSSOP-20_4.4x6.5mm_P0.65mm
- U5: footprint Housings_SSOP:TSSOP-24_4.4x7.8mm_Pitch0.65mm -> Package_SO:TSSOP-24_4.4x7.8mm_P0.65mm
- U7: footprint TO_SOT_Packages_SMD:SOT-23-5 -> Package_TO_SOT_SMD:SOT-23-5
Connections:
- wire segments 75 -> 72
- no-connect marks 10 -> 13
Other:
- note added: "SERCOM1 PAD 0"
- note added: "SERCOM5 PAD 0"
- moved on the sheet: R6, R7

Commit message: More work on v5
Parts:
- removed U3, U4, U6: 74LS244, Package_SO:TSSOP-20_4.4x6.5mm_P0.65mm, symbol pygameboy-rescue:74LS244-Logic_74xx
- added R8: 470, Resistor_SMD:R_0603_1608Metric_Pad1.05x0.95mm_HandSolder, symbol Device:R_Small
- added U3, U4, U6: 74LVC244, Package_SO:TSSOP-20_4.4x6.5mm_P0.65mm, symbol 74xx:74HC244
- C14: footprint Capacitor_SMD:C_0603_1608Metric_Pad1.05x0.95mm_HandSolder -> Capacitor_SMD:C_0805_2012Metric_Pad1.15x1.40mm_HandSolder
- D3: footprint LED_SMD:LED_0603_1608Metric_Pad1.05x0.95mm_HandSolder -> LED_SMD:LED_0805_2012Metric_Pad1.15x1.40mm_HandSolder
- U2: footprint Package_QFP:LQFP-64_10x10mm_P0.5mm -> Package_DFN_QFN:QFN-64-1EP_9x9mm_P0.5mm_EP4.7x4.7mm_ThermalVias; symbol pygameboy-rescue:SAMD51J-atmel-sam -> atmel-sam:SAMD51J
Connections:
- wire segments 72 -> 75
Changed lines of the file:
@@
 $EndDescr
 $Comp
-L pygameboy-rescue:SAMD51J-atmel-sam U2
+L atmel-sam:SAMD51J U2
 U 1 1 5AD3C3C3
 P 6400 3875
 F 0 "U2" H 6350 4000 60  0000 L CNN
 F 1 "SAMD51J" H 6250 3850 60  0000 L CNN
-F 2 "Package_QFP:LQFP-64_10x10mm_P0.5mm" H 6400 3875 60  0001 C CNN
+F 2 "Package_DFN_QFN:QFN-64-1EP_9x9mm_P0.5mm_EP4.7x4.7mm_ThermalVias" H 6400 3875 60  0001 C CNN
 F 3 "" H 6400 3875 60  0001 C CNN
 	1    6400 3875
-	1    0    0    -1
-$EndComp
-$Comp
-L pygameboy-rescue:74LS244-Logic_74xx U3
-U 1 1 5AD44766
-P 2925 4200
-F 0 "U3" H 2925 4450 50  0000 C CNN
-F 1 "74LS244" H 2925 3900 50  0000 C CNN
-F 2 "Package_SO:TSSOP-20_4.4x6.5mm_P0.65mm" H 2925 4200 50  0001 C CNN
-F 3 "http://www.ti.com/lit/gpn/sn74LS244" H 2925 4200 50  0001 C CNN
-	1    2925 4200
-	1    0    0    -1
-$EndComp
-$Comp
-L pygameboy-rescue:74LS244-Logic_74xx U4
-U 1 1 5AD447DE
-P 4425 3050
-F 0 "U4" H 4425 3250 50  0000 C CNN
-F 1 "74LS244" H 4425 2725 50  0000 C CNN
-F 2 "Package_SO:TSSOP-20_4.4x6.5mm_P0.65mm" H 4425 3050 50  0001 C CNN
-F 3 "http://www.ti.com/lit/gpn/sn74LS244" H 4425 3050 50  0001 C CNN
-	1    4425 3050
 	1    0    0    -1
 $EndComp
@@
 	1    1375 2825
 	0    1    1    0
-$EndComp
-$Comp
-L pygameboy-rescue:74LS244-Logic_74xx U6
-U 1 1 5AE766D2
-P 3075 1700
-F 0 "U6" H 3075 1950 50  0000 C CNN
-F 1 "74LS244" H 3075 1400 50  0000 C CNN
-F 2 "Package_SO:TSSOP-20_4.4x6.5mm_P0.65mm" H 3075 1700 50  0001 C CNN
-F 3 "http://www.ti.com/lit/gpn/sn74LS244" H 3075 1700 50  0001 C CNN
-	1    3075 1700
-	1    0    0    -1
 $EndComp
 $Comp
@@
 Text Label 2575 1900 2    50   ~ 0
 A3
+Text Label 3925 2850 2    50   ~ 0
+A4
+Text Label 3925 2750 2    50   ~ 0
+A5
+Text Label 3925 2650 2    50   ~ 0
+A6
 Text Label 3925 2550 2    50   ~ 0
-A4
-Text Label 3925 2650 2    50   ~ 0
-A5
-Text Label 3925 2750 2    50   ~ 0
-A6
-Text Label 3925 2850 2    50   ~ 0
 A7
+Text Label 3925 3250 2    50   ~ 0
+A8
+Text Label 3925 3150 2    50   ~ 0
+A9
+Text Label 3925 3050 2    50   ~ 0
+A10
 Text Label 3925 2950 2    50   ~ 0
-A8
-Text Label 3925 3050 2    50   ~ 0
-A9
-Text Label 3925 3150 2    50   ~ 0
-A10
-Text Label 3925 3250 2    50   ~ 0
 A11
 Text Label 2425 3700 2    50   ~ 0
@@
 Wire Wire Line
 	2575 2200 2425 2200
-Connection ~ 2575 2200
 Wire Wire Line
 	3925 3450 3925 3550
@@
 Text Label 5650 2525 1    50   ~ 0
 3V_A3
+Text Label 4925 2850 0    50   ~ 0
+3V_A4
+Text Label 4925 2750 0    50   ~ 0
+3V_A5
+Text Label 4925 2650 0    50   ~ 0
+3V_A6
 Text Label 4925 2550 0    50   ~ 0
-3V_A4
-Text Label 4925 2650 0    50   ~ 0
-3V_A5
-Text Label 4925 2750 0    50   ~ 0
-3V_A6
-Text Label 4925 2850 0    50   ~ 0
 3V_A7
+Text Label 4925 3250 0    50   ~ 0
+3V_A8
+Text Label 4925 3150 0    50   ~ 0
+3V_A9
+Text Label 4925 3050 0    50   ~ 0
+3V_A10
 Text Label 4925 2950 0    50   ~ 0
-3V_A8
-Text Label 4925 3050 0    50   ~ 0
-3V_A9
-Text Label 4925 3150 0    50   ~ 0
-3V_A10
-Text Label 4925 3250 0    50   ~ 0
 3V_A11
 Text Label 3425 3700 0    50   ~ 0
@@
 F 0 "D3" V 8438 2083 50  0000 R CNN
 F 1 "LED" V 8347 2083 50  0000 R CNN
-F 2 "LED_SMD:LED_0603_1608Metric_Pad1.05x0.95mm_HandSolder" H 8400 2200 50  0001 C CNN
+F 2 "LED_SMD:LED_0805_2012Metric_Pad1.15x1.40mm_HandSolder" H 8400 2200 50  0001 C CNN
 F 3 "~" H 8400 2200 50  0001 C CNN
 	1    8400 2200
@@
 F 0 "C14" V 6750 1850 50  0000 C CNN
 F 1 "10uF" V 6825 1850 50  0000 C CNN
-F 2 "Capacitor_SMD:C_0603_1608Metric_Pad1.05x0.95mm_HandSolder" H 6950 1850 50  0001 C CNN
+F 2 "Capacitor_SMD:C_0805_2012Metric_Pad1.15x1.40mm_HandSolder" H 6950 1850 50  0001 C CNN
 F 3 "" H 6950 1850 50  0001 C CNN
 	1    6950 1850
@@
 	1    0    0    -1
 $EndComp
-Text Label 10575 3875 0    50   ~ 0
+Text Label 10800 3875 0    50   ~ 0
 MIDI_IN
 $Comp
@@
 Wire Wire Line
 	10700 3575 10275 3575
-Text Label 5400 3125 1    50   ~ 0
+Text Label 5400 3125 2    50   ~ 0
 MIDI_IN
 Text Notes 6050 2175 1    50   ~ 0
@@
 NoConn ~ 9350 4550
 NoConn ~ 9350 4750
+$Comp
+L 74xx:74HC244 U4
+U 1 1 5C86A82C
+P 4425 3050
+F 0 "U4" H 4425 4028 50  0000 C CNN
+F 1 "74LVC244" H 4425 3937 50  0000 C CNN
+F 2 "Package_SO:TSSOP-20_4.4x6.5mm_P0.65mm" H 4425 3050 50  0001 C CNN
+F 3 "http://www.nxp.com/documents/data_sheet/74HC_HCT244.pdf" H 4425 3050 50  0001 C CNN
+	1    4425 3050
+	1    0    0    -1
+$EndComp
+$Comp
+L 74xx:74HC244 U6
+U 1 1 5C845FB0
+P 3075 1700
+F 0 "U6" H 3075 2678 50  0000 C CNN
+F 1 "74LVC244" H 3075 2587 50  0000 C CNN
+F 2 "Package_SO:TSSOP-20_4.4x6.5mm_P0.65mm" H 3075 1700 50  0001 C CNN
+F 3 "http://www.nxp.com/documents/data_sheet/74HC_HCT244.pdf" H 3075 1700 50  0001 C CNN
+	1    3075 1700
+	1    0    0    -1
+$EndComp
+Connection ~ 2575 2200
+$Comp
+L 74xx:74HC244 U3
+U 1 1 5C84622A
+P 2925 4200
+F 0 "U3" H 2925 5178 50  0000 C CNN
+F 1 "74LVC244" H 2925 5087 50  0000 C CNN
+F 2 "Package_SO:TSSOP-20_4.4x6.5mm_P0.65mm" H 2925 4200 50  0001 C CNN
+F 3 "http://www.nxp.com/documents/data_sheet/74HC_HCT244.pdf" H 2925 4200 50  0001 C CNN
+	1    2925 4200
+	1    0    0    -1
+$EndComp
+$Comp
+L power:GND #PWR0165
+U 1 1 5C849BE4
+P 5400 3025
+F 0 "#PWR0165" H 5400 2775 50  0001 C CNN
+F 1 "GND" H 5405 2852 50  0000 C CNN
+F 2 "" H 5400 3025 50  0001 C CNN
+F 3 "" H 5400 3025 50  0001 C CNN
+	1    5400 3025
+	-1   0    0    1
+$EndComp
+$Comp
+L Device:R_Small R8
+U 1 1 5C84EA32
+P 10700 3675
+F 0 "R8" H 10759 3721 50  0000 L CNN
+F 1 "470" H 10759 3630 50  0000 L CNN
+F 2 "Resistor_SMD:R_0603_1608Metric_Pad1.05x0.95mm_HandSolder" H 10700 3675 50  0001 C CNN
+F 3 "~" H 10700 3675 50  0001 C CNN
+	1    10700 3675
+	1    0    0    -1
+$EndComp
+Wire Wire Line
+	10575 3875 10700 3875
+Wire Wire Line
+	10700 3775 10700 3875
+Connection ~ 10700 3875
+Wire Wire Line
+	10700 3875 10800 3875
 $EndSCHEMATC

Commit message: Final v5 version
Parts:
- added FID0, FID1: TestPoint, Fiducial:Fiducial_1mm_Mask2mm, symbol Connector:TestPoint
- added TP48, TP49, TP50, TP51, TP52, TP53, TP54, TP55, TP56, TP57, TP58, TP59, TP60, TP61, TP62, TP63, TP64, TP65, TP66, TP67, TP68, TP69, TP70, TP71, TP72, TP73, TP74, TP75, TP76, TP77, TP78, TP79, TP80, TP81, TP82, TP83, TP84, TP85: Test_Point, TestPoint:TestPoint_Pad_D1.5mm, symbol pygameboy-rescue:Test_Point-Connector
Connections:
- net labels added: AUD
- no-connect marks 13 -> 12
Other:
- note added: "Bottom test points\nfor test jig"
- note added: "Fiducials"
- moved on the sheet: U1

Commit message: Correct optoistolator footprint. Tweak spacing.
Parts:
- J3: symbol Connector:Conn_ARM_JTAG_SWD_10 -> pygameboy-rescue:Conn_ARM_JTAG_SWD_10-Connector
- U8: footprint Package_DIP:SMDIP-6_W7.62mm -> Package_DIP:SMDIP-6_W9.53mm
Changed lines of the file:
@@
 EESchema Schematic File Version 4
 LIBS:pygameboy-cache
-EELAYER 26 0
+EELAYER 29 0
 EELAYER END
 $Descr A4 11693 8268
@@
 3V_D0
 $Comp
-L Connector:Conn_ARM_JTAG_SWD_10 J3
+L pygameboy-rescue:Conn_ARM_JTAG_SWD_10-Connector J3
 U 1 1 5AE826AA
 P 7675 1300
@@
 F 0 "U8" H 10525 3700 50  0000 L CNN
 F 1 "H11L1" H 10525 3775 50  0000 L CNN
-F 2 "Package_DIP:SMDIP-6_W7.62mm" H 10185 3875 50  0001 C CNN
+F 2 "Package_DIP:SMDIP-6_W9.53mm" H 10185 3875 50  0001 C CNN
 F 3 "https://www.fairchildsemi.com/datasheets/H1/H11L1M.pdf" H 10185 3875 50  0001 C CNN
 	1    10275 3875
@@
 $EndComp
 $Comp
-L power:GND #PWR?
+L power:GND #PWR0169
 U 1 1 5C87942F
 P 10600 1725
-F 0 "#PWR?" H 10600 1475 50  0001 C CNN
+F 0 "#PWR0169" H 10600 1475 50  0001 C CNN
 F 1 "GND" H 10605 1552 50  0000 C CNN
 F 2 "" H 10600 1725 50  0001 C CNN

Commit message: Update for kicad 5.1.6 and use submodule for kicad-libs
Parts:
- C1, C11, C12, C13, C14, C15, C2, C3, C4, C5, C6, C7, C9: symbol pygameboy-rescue:C_Small-device -> Device:C_Small
- D1, D2: symbol pygameboy-rescue:D_Schottky-device -> Device:D_Schottky
- D3: symbol pygameboy-rescue:LED-device -> Device:LED
- J1, J2: symbol pygameboy-rescue:Conn_01x01-Connector -> Connector_Generic:Conn_01x01
- J3: symbol pygameboy-rescue:Conn_ARM_JTAG_SWD_10-Connector -> Connector:Conn_ARM_JTAG_SWD_10
- Q1: symbol pygameboy-rescue:BSS138-Transistor -> Transistor_FET:BSS138
- R1, R2, R3, R4: symbol pygameboy-rescue:R_Small-device -> Device:R_Small
- TP1, TP10, TP11, TP12, TP13, TP14, TP15, TP16, TP17, TP18, TP19, TP2, TP20, TP21, TP22, TP23, TP24, TP25, TP26, TP27, TP28, TP29, TP3, TP30, TP31, TP32, TP33, TP34, TP35, TP36, TP37, TP38, TP39, TP4, TP40, TP41, TP42, TP43, TP44, TP45, TP46, TP47, TP48, TP49, TP5, TP50, TP51, TP52, TP53, TP54, TP55, TP56, TP57, TP58, TP59, TP6, TP60, TP61, TP62, TP63, TP64, TP65, TP66, TP67, TP68, TP69, TP7, TP70, TP71, TP72, TP73, TP74, TP75, TP76, TP77, TP78, TP79, TP8, TP80, TP81, TP82, TP83, TP84, TP85, TP9: symbol pygameboy-rescue:Test_Point-Connector -> Connector:TestPoint
- U7: symbol pygameboy-rescue:AP2204K-3.3-regul -> Regulator_Linear:AP2204K-3.3
Connections:
- wire segments 75 -> 73

Commit message: Start of breakout version
Parts:
- removed C1, C2, C3, C4, C5, C6: 0.1uF, Capacitor_SMD:C_0603_1608Metric_Pad1.05x0.95mm_HandSolder, symbol Device:C_Small
- removed C10, C13, C15: 1uF, Capacitor_SMD:C_0603_1608Metric_Pad1.05x0.95mm_HandSolder, symbol Device:C_Small
- removed C14: 10uF, Capacitor_SMD:C_0805_2012Metric_Pad1.15x1.40mm_HandSolder, symbol Device:C_Small
- removed C16, C17: C_Small, Capacitor_SMD:C_0603_1608Metric_Pad1.05x0.95mm_HandSolder, symbol Device:C_Small
- removed D1, D2: MBR120, Diode_SMD:D_SOD-123, symbol Device:D_Schottky
- removed D4: 1N4148W, Diode_SMD:D_SOD-123, symbol Diode:1N4148W
- removed J3: Conn_ARM_JTAG_SWD_10, Pin_Headers:Pin_Header_Straight_2x05_Pitch1.27mm_SMD, symbol Connector:Conn_ARM_JTAG_SWD_10
- removed J4: USB_B_Micro, adafruit:4UCONN_20329_V2_USB, symbol Connector:USB_B_Micro
- removed J5: MIDI IN, adafruit:4UCONN_19269_TRS, symbol Connector:AudioJack3_SwitchTR
- removed J6: MIDI OUT, adafruit:4UCONN_19269_TRS, symbol Connector:AudioJack3_SwitchTR
- removed R1: 10k, Resistor_SMD:R_0603_1608Metric_Pad1.05x0.95mm_HandSolder, symbol Device:R_Small
- removed R5: 220, Resistor_SMD:R_0603_1608Metric_Pad1.05x0.95mm_HandSolder, symbol Device:R_Small
- removed R6, R7: 51, Resistor_SMD:R_0603_1608Metric_Pad1.05x0.95mm_HandSolder, symbol Device:R_Small
- removed R8: 470, Resistor_SMD:R_0603_1608Metric_Pad1.05x0.95mm_HandSolder, symbol Device:R_Small
- removed SW1: SW_Push, Button_Switch_SMD:SW_SPST_KMR2, symbol Switch:SW_Push
- removed TP33: Test_Point, keystone:5015-SMT-TestPoint, symbol Connector:TestPoint
- removed TP34: DATA_OE, keystone:5015-SMT-TestPoint, symbol Connector:TestPoint
- removed TP35: GB_RESET, keystone:5015-SMT-TestPoint, symbol Connector:TestPoint
- removed TP36: SAMD_RESET, keystone:5015-SMT-TestPoint, symbol Connector:TestPoint
- removed TP40: clk, keystone:5015-SMT-TestPoint, symbol Connector:TestPoint
- removed TP41: rd, keystone:5015-SMT-TestPoint, symbol Connector:TestPoint
- removed TP42: wr, keystone:5015-SMT-TestPoint, symbol Connector:TestPoint
- removed TP43: a15, keystone:5015-SMT-TestPoint, symbol Connector:TestPoint
- removed TP44: PB17, keystone:5015-SMT-TestPoint, symbol Connector:TestPoint
- removed TP45: cs, keystone:5015-SMT-TestPoint, symbol Connector:TestPoint
- removed TP46: data0, keystone:5015-SMT-TestPoint, symbol Connector:TestPoint
- removed TP47: D0, keystone:5015-SMT-TestPoint, symbol Connector:TestPoint
- removed TP80, TP81, TP82, TP83, TP84, TP85: Test_Point, TestPoint:TestPoint_Pad_D1.5mm, symbol Connector:TestPoint
- removed U2: SAMD51J, Package_DFN_QFN:QFN-64-1EP_9x9mm_P0.5mm_EP4.7x4.7mm_ThermalVias, symbol atmel-sam:SAMD51J
- removed U7: AP2204K-3.3, Package_TO_SOT_SMD:SOT-23-5, symbol Regulator_Linear:AP2204K-3.3
- removed U8: H11L1, Package_DIP:SMDIP-6_W9.53mm, symbol Isolator:H11L1
- added J3, J4, J5, J6: Conn_02x05_Odd_Even, adafruit:PinHeader_2x05_P1.27mm_Vertical_SMD, symbol Connector_Generic:Conn_02x05_Odd_Even
Connections:
- net labels removed: +BATT, LED, MIDI_IN, MIDI_OUT, SAMD_RESET, SHIELD, SWCLK, SWDIO, SWO, USB_D+, USB_D-, VBUS
- wire segments 73 -> 21
- no-connect marks 12 -> 6
Other:
- note removed: "SERCOM1 PAD 0"
- note removed: "SERCOM5 PAD 0"
- moved on the sheet: D3, R4
