File: pygameboy.sch (KiCad schematic (older format))
At the start: 132 parts, among them J1 Conn_01x01, J2 Conn_01x01, J3 Conn_ARM_JTAG_SWD_10, J4 USB_B_Micro, J5 MIDI IN, J6 MIDI OUT, Q1 BSS138, SW1 SW_Push, U1 CARTRIDGE, U2 SAMD51J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

Commit message: rp2040 start
Parts:
- removed TP44: PB17, keystone:5015-SMT-TestPoint, symbol Connector:TestPoint
- removed U2: SAMD51J, Package_DFN_QFN:QFN-64-1EP_9x9mm_P0.5mm_EP4.7x4.7mm_ThermalVias, symbol atmel-sam:SAMD51J
- added C18, C20, C21, C22: 0.1uF, Capacitor_SMD:C_0603_1608Metric_Pad1.08x0.95mm_HandSolder, symbol Device:C_Small
- added C19: 1uF, Capacitor_SMD:C_0603_1608Metric_Pad1.08x0.95mm_HandSolder, symbol Device:C_Small
- added R10: 1k, Resistor_SMD:R_0603_1608Metric_Pad0.98x0.95mm_HandSolder, symbol Device:R_Small
- added R11, R12: 27, Resistor_SMD:R_0603_1608Metric_Pad0.98x0.95mm_HandSolder, symbol Device:R_Small
- added R9: 10k, Resistor_SMD:R_0603_1608Metric_Pad0.98x0.95mm_HandSolder, symbol Device:R_Small
- added U2: RP2040, MCU_RaspberryPi_and_Boards:RP2040-QFN-56, symbol MCU_RaspberryPi_and_Boards:RP2040
- added U9: W25Q32JVSS, Package_SO:SOIC-8_5.23x5.23mm_P1.27mm, symbol Memory_Flash:W25Q32JVSS
- added Y1: 12mhz, Crystal:Crystal_SMD_Abracon_ABM3C-4Pin_5.0x3.2mm, symbol Device:Crystal
- C1, C2: value 0.1uF -> 22pF; footprint Capacitor_SMD:C_0603_1608Metric_Pad1.05x0.95mm_HandSolder -> Capacitor_SMD:C_0402_1005Metric_Pad0.74x0.62mm_HandSolder
- C10, C11, C12, C13, C16, C17, C3, C5, C6, C7, C8, C9: footprint Capacitor_SMD:C_0603_1608Metric_Pad1.05x0.95mm_HandSolder -> Capacitor_SMD:C_0603_1608Metric_Pad1.08x0.95mm_HandSolder
- C14: value 10uF -> 0.1uF; footprint Capacitor_SMD:C_0805_2012Metric_Pad1.15x1.40mm_HandSolder -> Capacitor_SMD:C_0603_1608Metric_Pad1.08x0.95mm_HandSolder
- C15: value 1uF -> 0.1uF; footprint Capacitor_SMD:C_0603_1608Metric_Pad1.05x0.95mm_HandSolder -> Capacitor_SMD:C_0603_1608Metric_Pad1.08x0.95mm_HandSolder
- C4: value 0.1uF -> 1uF; footprint Capacitor_SMD:C_0603_1608Metric_Pad1.05x0.95mm_HandSolder -> Capacitor_SMD:C_0603_1608Metric_Pad1.08x0.95mm_HandSolder
- R1, R2, R3, R4, R5, R6, R7, R8: footprint Resistor_SMD:R_0603_1608Metric_Pad1.05x0.95mm_HandSolder -> Resistor_SMD:R_0603_1608Metric_Pad0.98x0.95mm_HandSolder
Connections:
- net labels added: QSPI_CS, QSPI_SCLK, QSPI_SD0, QSPI_SD1, QSPI_SD2, QSPI_SD3
- net labels removed: DIR
- wire segments 73 -> 105
Other:
- note removed: "SERCOM1 PAD 0"
- note removed: "SERCOM5 PAD 0"
- moved on the sheet: C10, C12, C13, C16, D1, D2, D3, J3, Q1, R1, R2, R3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
