File: pygameboy.kicad_pcb (KiCad board)
At the start: 2 copper layers, 49.3 x 59.7 mm, 90 parts, among them J1 Conn_01x01, J2 Conn_01x01, J3 Conn_02x05_Odd_Even, J4 Conn_02x05_Odd_Even, J5 Conn_02x05_Odd_Even, J6 Conn_02x05_Odd_Even, Q1 BSS138, U1 CARTRIDGE, U3 74LVC244, U4 74LVC244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

Commit message: v1
Parts:
- added G***: Chickadee 3mm, chickadee:chickadee_3mm_fcu, F.Cu at (123.0, 60.3)
- moved R3 21.5 mm to (127.9, 42.0), turned to 270 degrees
Routing:
- net +3V3: track 59.2 -> 197.0 mm, vias 4 -> 18
- net +5V: track 27.0 -> 89.0 mm, vias 1 -> 2
- net /AUD: track 19.0 -> 80.6 mm, vias 1 -> 6
- net /GB_RESET: track 7.39 -> 40.9 mm, vias 1 -> 4
- net /DATA_OE: track 57.4 -> 45.5 mm, vias 2 -> 0
- net /3V_A10: track 46.8 -> 39.0 mm
- net GND: track 82.7 -> 89.3 mm, vias 18 -> 19
- net /DIR: track 47.6 -> 45.1 mm
- net /3V_A8: track 47.8 -> 50.2 mm
- net /3V_A9: track 44.7 -> 46.9 mm
- net /3V_A7: track 48.9 -> 47.9 mm
- net /3V_CLK: track 35.7 -> 36.6 mm
- net /3V_RD: track 32.5 -> 31.7 mm
- net /3V_A6: track 45.2 -> 44.5 mm
- net /3V_A11: track 48.0 -> 47.3 mm
Other:
- board text added: "3.3V"
- board text added: "A0-A7"
- board text added: "A8-A15"
- board text added: "CONTROL"
- board text added: "D0-D7"
- board text added: "PWR"
- board text added: "ckd.tech/gb-bo/v1"
- board text removed: "LED"
- board text removed: "ckd.tech/pygb/v6"
