File: rp2350.kicad_sch (KiCad schematic)
At the start: 30 parts, among them U10 RP2350_80QFN, U2 W25Q128JVS, Y1 ABM8-272-T3

Commit message: Ordered!
Parts:
- removed R10: 0, Resistor_SMD:R_0402_1005Metric, symbol Device:R
- removed R9: DNF, Resistor_SMD:R_0402_1005Metric, symbol Device:R
- R201: renamed from R12; value DNF -> 10k
- renumbered C1 to C201, C3 to C202, C4 to C203, C5 to C204, C6 to C205, C11 to C206, C14 to C207, C15 to C208, C18 to C209, C19 to C210, C20 to C211, C21 to C212, C22 to C213, C23 to C214, C24 to C215, C25 to C216, C26 to C217, C27 to C218, L1 to L201, R14 to R202, R15 to R203, R16 to R204, R17 to R205, R18 to R206, U2 to U201, U10 to U202, Y1 to Y201
Connections:
- net FLASH_SS is gone; now on net QSPI_SS: R201.2, U201.1 (~{CS})
- net GND: now also R204.2
- net RUN: now also U202.35 (RUN)
Other:
- moved on the sheet: C201, R201, U201

Commit message: Fix reset circuit. Move control signals to higher pins that both PIO offsets can read. Redo audio circuit
Connections:
- net GND: no longer R204.2
- new net BOOT: R204.2
Changed lines of the file:
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@@
 	(wire
 		(pts
-			(xy 96.52 92.71) (xy 102.87 92.71)
-		)
-		(stroke
-			(width 0)
-			(type default)
-		)
-	)
-	(wire
-		(pts
 			(xy 215.9 16.51) (xy 215.9 15.24)
 		)
@@
 		)
 	)
-	(label "QSPI_SS"
-		(at 102.87 92.71 0)
-		(effects
-			(font
-				(size 1.27 1.27)
-			)
-			(justify left bottom)
-		)
-	)
 	(label "XIN"
 		(at 111.76 179.705 180)
@@
 		)
 	)
+	(hierarchical_label "BOOT"
+		(shape input)
+		(at 118.11 77.47 180)
+		(effects
+			(font
+				(size 1.27 1.27)
+			)
+			(justify right)
+		)
+	)
 	(hierarchical_label "GPIO16"
 		(shape input)
@@
 		)
 	)
-	(hierarchical_label "QSPI_SS"
-		(shape input)
-		(at 96.52 92.71 180)
-		(effects
-			(font
-				(size 1.27 1.27)
-			)
-			(justify right)
-		)
-	)
 	(hierarchical_label "GPIO13"
 		(shape input)
@@
 					(unit 1)
 				)
-			)
-		)
-	)
-	(symbol
-		(lib_id "power:GND")
-		(at 118.11 77.47 0)
-		(unit 1)
-		(body_style 1)
-		(exclude_from_sim no)
-		(in_bom yes)
-		(on_board yes)
-		(in_pos_files yes)
-		(dnp no)
-		(property "Reference" "#PWR0210"
-			(at 118.11 83.82 0)
-			(hide yes)
-			(show_name no)
-			(do_not_autoplace no)
-			(effects
-				(font
-					(size 1.27 1.27)
-				)
-			)
-		)
-		(property "Value" "GND"
-			(at 118.237 81.8642 0)
-			(show_name no)
-			(do_not_autoplace no)
-			(effects
-				(font
-					(size 1.27 1.27)
-				)
-			)
-		)
-		(property "Footprint" ""
-			(at 118.11 77.47 0)
-			(hide yes)
-			(show_name no)
-			(do_not_autoplace no)
-			(effects
-				(font
-					(size 1.27 1.27)
-				)
-			)
-		)
-		(property "Datasheet" ""
-			(at 118.11 77.47 0)
-			(hide yes)
-			(show_name no)
-			(do_not_autoplace no)
-			(effects
-				(font
-					(size 1.27 1.27)
-				)
-			)
-		)
-		(property "Description" ""
-			(at 118.11 77.47 0)
-			(show_name no)
-			(do_not_autoplace no)
-			(effects
-				(font
-					(size 1.27 1.27)
-				)
-			)
-		)
-		(pin "1"
-		)
-		(instances
-			(project "pygameboy"
-				(path "/63efa618-1458-4f61-941c-03fd363e3bea/e20e6721-8f13-4e3b-9d71-8094fcd7542f"
-					(reference "#PWR0210")
-					(unit 1)
-				)
