File: rp2350.kicad_sch (KiCad schematic)
At the start: 28 parts, among them U201 W25Q128JVS, U202 RP2350_80QFN, Y201 ABM8-272-T3

Commit message: WIP v9
Parts:
- added D201: 1N4148W, Diode_SMD:D_SOD-123, symbol Diode:1N4148W
- C207, C208: footprint Capacitor_SMD:C_0402_1005Metric -> Capacitor_SMD:C_0805_2012Metric
Connections:
- net BOOT: now also D201.1 (K); no longer R204.2
- new net: D201.2 (A), R204.2
Other:
- note added: "TODO: Add PSRAM footprint if we have space. C3040877 8MB APS USON-L SOP-8"
Changed lines of the file:
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@@
 		)
 	)
+	(text "TODO: Add PSRAM footprint if we have space.\nC3040877 8MB APS USON-L SOP-8"
+		(exclude_from_sim no)
+		(at 86.614 99.06 0)
+		(effects
+			(font
+				(size 1.27 1.27)
+			)
+		)
+	)
 	(junction
 		(at 95.25 69.85)
@@
 		)
 	)
+	(label "NEOPIXEL"
+		(at 2.6988 4.5468 0)
+		(effects
+			(font
+				(size 1.27 1.27)
+			)
+			(justify left bottom)
+		)
+	)
 	(label "QSPI_SD1"
 		(at 73.025 80.01 180)
@@
 		)
 	)
+	(hierarchical_label "SWD"
+		(shape input)
+		(at 128.27 133.35 180)
+		(effects
+			(font
+				(size 1.27 1.27)
+			)
+			(justify right)
+		)
+	)
 	(hierarchical_label "GPIO30"
 		(shape input)
@@
 	(hierarchical_label "BOOT"
 		(shape input)
-		(at 118.11 77.47 180)
+		(at 110.49 77.47 180)
 		(effects
 			(font
@@
 		)
 	)
+	(hierarchical_label "SWCLK"
+		(shape input)
+		(at 128.27 130.81 180)
+		(effects
+			(font
+				(size 1.27 1.27)
+			)
+			(justify right)
+		)
+	)
 	(hierarchical_label "GPIO6"
 		(shape input)
@@
 	)
 	(symbol
+		(lib_id "Diode:1N4148W")
+		(at 114.3 77.47 0)
+		(mirror x)
+		(unit 1)
+		(body_style 1)
+		(exclude_from_sim no)
+		(in_bom yes)
+		(on_board yes)
+		(in_pos_files yes)
+		(dnp no)
+		(property "Reference" "D201"
+			(at 113.1316 79.502 90)
+			(show_name no)
+			(do_not_autoplace no)
+			(effects
+				(font
+					(size 1.27 1.27)
+				)
+				(justify left)
+			)
+		)
+		(property "Value" "1N4148W"
+			(at 115.57 79.756 90)
+			(show_name no)
+			(do_not_autoplace no)
+			(effects
+				(font
+					(size 1.27 1.27)
+				)
+				(justify left)
+			)
+		)
+		(property "Footprint" "Diode_SMD:D_SOD-123"
+			(at 114.3 73.025 0)
+			(hide yes)
+			(show_name no)
+			(do_not_autoplace no)
+			(effects
+				(font
+					(size 1.27 1.27)
+				)
+			)
+		)
+		(property "Datasheet" "https://www.vishay.com/docs/85748/1n4148w.pdf"
+			(at 114.3 77.47 0)
+			(hide yes)
+			(show_name no)
+			(do_not_autoplace no)
+			(effects
+				(font
+					(size 1.27 1.27)
+				)
+			)
+		)
+		(property "Description" ""
+			(at 114.3 77.47 0)
+			(hide yes)
+			(show_name no)
+			(do_not_autoplace no)
+			(effects
+				(font
+					(size 1.27 1.27)
+				)
+			)
+		)
+		(pin "1"
+		)
+		(pin "2"
+		)
+		(instances
+			(project "pygameboy"
+				(path "/63efa618-1458-4f61-941c-03fd363e3bea/e20e6721-8f13-4e3b-9d71-8094fcd7542f"
+					(reference "D201")
+					(unit 1)
+				)
+			)
+		)
+	)
+	(symbol
 		(lib_id "Device:C")
 		(at 215.9 20.32 0)
@@
 			)
 		)
-		(property "Footprint" "Capacitor_SMD:C_0402_1005Metric"
+		(property "Footprint" "Capacitor_SMD:C_0805_2012Metric"
 			(at 130.5052 53.34 0)
 			(hide yes)
@@
 			)
 		)
-		(property "Footprint" "Capacitor_SMD:C_0402_1005Metric"
+		(property "Footprint" "Capacitor_SMD:C_0805_2012Metric"
 			(at 131.7752 24.13 0)
 			(hide yes)

Commit message: Half routed. microsd added
Parts:
- added C219: 100n, Capacitor_SMD:C_0402_1005Metric, symbol Device:C
- added R208: 10k, Resistor_SMD:R_0402_1005Metric, symbol Device:R
- added U203: APS6404L-3SQR-ZR, Package_SO:SOP-8_3.76x4.96mm_P1.27mm, symbol Memory_Flash:W25Q128JVS
- D201: footprint Diode_SMD:D_SOD-123 -> Diode_SMD:D_SOD-523
Connections:
- net +3V3: now also C219.1, R208.1, U203.8 (VCC)
- net GND: now also C219.2, U203.4 (GND)
- net GPIO0: now also R208.2, U203.1 (~{CS})
- net QSPI_SCLK: now also U203.6 (CLK)
- net QSPI_SD0: now also U203.5 (DI(IO0))
- net QSPI_SD1: now also U203.2 (DO(IO1))
- net QSPI_SD2: now also U203.3 (IO2)
- net QSPI_SD3: now also U203.7 (IO3)
Other:
- note added: "For PSRAM"
- note added: "Secondary Flash/PSRAM"
