File: pygameboy.kicad_sch (KiCad schematic)
At the start: 105 parts, among them J1 Conn_01x01, J14 Conn_01x04, J2 Conn_01x01, J4 USB_C_Receptacle_USB2.0_16P, J5 AudioJack4, J6 AudioJack4, Q1 BSS138, SW1 SW_Push, SW2 SW_Push, U1 CARTRIDGE, U5 74x4245, U7 AP2204K-3.3, U8 H11L1

Commit message: Update to v8
Parts:
- added J101: Conn_01x03, Connector_JST:JST_SH_BM03B-SRSS-TB_1x03-1MP_P1.00mm_Vertical, symbol Connector_Generic:Conn_01x03
Connections:
- net GND: now also J101.2 (Pin_2)
- new net DEBUG_RX: J101.1 (Pin_1)
- new net DEBUG_TX: J101.3 (Pin_3)
- no-connect marks 9 -> 4
Changed lines of the file:
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@@
 	)
 	(no_connect
-		(at 173.99 121.92)
-	)
-	(no_connect
 		(at 247.65 60.96)
 	)
 	(no_connect
-		(at 179.07 121.92)
-	)
-	(no_connect
 		(at 156.845 26.035)
 	)
 	(no_connect
-		(at 181.61 121.92)
-	)
-	(no_connect
 		(at 156.845 19.05)
 	)
@@
 		(at 247.65 63.5)
 	)
-	(no_connect
-		(at 184.15 121.92)
-	)
-	(no_connect
-		(at 176.53 121.92)
-	)
 	(wire
 		(pts
@@
 	(wire
 		(pts
-			(xy 194.31 121.92) (xy 194.31 124.46)
+			(xy 179.07 121.92) (xy 179.07 124.46)
 		)
 		(stroke
@@
 	(wire
 		(pts
-			(xy 207.01 113.03) (xy 209.55 113.03)
+			(xy 191.77 121.92) (xy 191.77 124.46)
 		)
 		(stroke
@@
 	(wire
 		(pts
-			(xy 196.85 121.92) (xy 196.85 124.46)
+			(xy 181.61 121.92) (xy 181.61 124.46)
 		)
 		(stroke
@@
 	(wire
 		(pts
-			(xy 191.77 121.92) (xy 191.77 124.46)
+			(xy 176.53 121.92) (xy 176.53 124.46)
 		)
 		(stroke
@@
 	(wire
 		(pts
-			(xy 186.69 121.92) (xy 186.69 124.46)
+			(xy 171.45 121.92) (xy 171.45 124.46)
 		)
 		(stroke
@@
 	(wire
 		(pts
-			(xy 189.23 121.92) (xy 189.23 124.46)
+			(xy 173.99 121.92) (xy 173.99 124.46)
 		)
 		(stroke
@@
 	(wire
 		(pts
-			(xy 207.01 115.57) (xy 209.55 115.57)
+			(xy 189.23 121.92) (xy 189.23 124.46)
 		)
 		(stroke
@@
 	(wire
 		(pts
-			(xy 207.01 110.49) (xy 209.55 110.49)
+			(xy 194.31 121.92) (xy 194.31 124.46)
 		)
 		(stroke
@@
 	(wire
 		(pts
-			(xy 207.01 120.65) (xy 209.55 120.65)
+			(xy 184.15 121.92) (xy 184.15 124.46)
 		)
 		(stroke
@@
 	(wire
 		(pts
-			(xy 207.01 118.11) (xy 209.55 118.11)
+			(xy 186.69 121.92) (xy 186.69 124.46)
 		)
 		(stroke
@@
 	)
 	(label "3V_D2"
-		(at 194.31 124.46 270)
+		(at 179.07 124.46 270)
 		(effects
 			(font
@@
 	)
 	(label "DATA_OE"
-		(at 186.69 124.46 270)
+		(at 171.45 124.46 270)
 		(effects
 			(font
@@
 		)
 	)
+	(label "DEBUG_RX"
+		(at 207.01 95.25 0)
+		(effects
+			(font
+				(size 1.27 1.27)
+			)
+			(justify left bottom)
+		)
+	)
 	(label "RD"
 		(at 25.4 29.845 0)
@@
 		)
 	)
+	(label "DEBUG_TX"
+		(at 207.01 97.79 0)
+		(effects
+			(font
+				(size 1.27 1.27)
+			)
+			(justify left bottom)
+		)
+	)
 	(label "D6"
 		(at 75.565 155.575 180)
@@
 	)
 	(label "3V_D4"
-		(at 209.55 120.65 0)
+		(at 184.15 124.46 270)
 		(effects
 			(font
 				(size 1.27 1.27)
 			)
-			(justify left bottom)
+			(justify right bottom)
 		)
 	)
@@
 		)
 	)
+	(label "DEBUG_RX"
+		(at 227.33 74.93 180)
+		(effects
+			(font
+				(size 1.27 1.27)
+			)
+			(justify right bottom)
+		)
+	)
 	(label "A5"
 		(at 25.4 47.625 0)
@@
 	)
 	(label "3V_D7"
-		(at 209.55 113.03 0)
+		(at 191.77 124.46 270)
 		(effects
 			(font
 				(size 1.27 1.27)
 			)
-			(justify left bottom)
+			(justify right bottom)
 		)
 	)
@@
 	)
 	(label "3V_D1"
-		(at 191.77 124.46 270)
+		(at 176.53 124.46 270)
 		(effects
 			(font
@@
 	)
 	(label "3V_D3"
-		(at 196.85 124.46 270)
+		(at 181.61 124.46 270)
 		(effects
 			(font
@@
 		)
 	)
+	(label "DEBUG_TX"
+		(at 227.33 80.01 180)
+		(effects
+			(font
+				(size 1.27 1.27)
+			)
+			(justify right bottom)
+		)
+	)
 	(label "D5"
 		(at 24.765 180.34 180)
@@
 	)
 	(label "3V_D0"
-		(at 189.23 124.46 270)
+		(at 173.99 124.46 270)
 		(effects
 			(font
@@
 	)
 	(label "3V_D6"
-		(at 209.55 115.57 0)
+		(at 189.23 124.46 270)
 		(effects
 			(font
 				(size 1.27 1.27)
 			)
-			(justify left bottom)
+			(justify right bottom)
 		)
 	)
@@
 	)
 	(label "3V_D5"
-		(at 209.55 118.11 0)
+		(at 186.69 124.46 270)
 		(effects
 			(font
 				(size 1.27 1.27)
 			)
-			(justify left bottom)
+			(justify right bottom)
 		)
 	)
@@
 	)
 	(label "RP_GB_RESET"
-		(at 209.55 110.49 0)
+		(at 194.31 124.46 270)
 		(effects
 			(font
 				(size 1.27 1.27)
 			)
-			(justify left bottom)
+			(justify right bottom)
 		)
 	)
@@
 	)
 	(symbol
+		(lib_id "pygameboy-rescue:GND-power")
+		(at 227.33 77.47 270)
+		(unit 1)
+		(body_style 1)
+		(exclude_from_sim no)
+		(in_bom yes)
+		(on_board yes)
+		(in_pos_files yes)
+		(dnp no)
+		(property "Reference" "#PWR0107"
+			(at 220.98 77.47 0)
+			(hide yes)
+			(show_name no)
+			(do_not_autoplace no)
+			(effects
+				(font
+					(size 1.27 1.27)
+				)
+			)
+		)
+		(property "Value" "GND"
+			(at 222.504 76.962 90)
+			(show_name no)
+			(do_not_autoplace no)
+			(effects
+				(font
+					(size 1.27 1.27)
+				)
+			)
+		)
+		(property "Footprint" ""
+			(at 227.33 77.47 0)
+			(hide yes)
+			(show_name no)
+			(do_not_autoplace no)
+			(effects
+				(font
+					(size 1.27 1.27)
+				)
+			)
+		)
+		(property "Datasheet" ""
+			(at 227.33 77.47 0)
+			(hide yes)
+			(show_name no)
+			(do_not_autoplace no)
+			(effects
+				(font
+					(size 1.27 1.27)
+				)
+			)
+		)
+		(property "Description" ""
+			(at 227.33 77.47 0)
+			(hide yes)
+			(show_name no)
+			(do_not_autoplace no)
+			(effects
+				(font
+					(size 1.27 1.27)
+				)
+			)
+		)
+		(pin "1"
+		)
+		(instances
+			(project "pygameboy"
+				(path "/63efa618-1458-4f61-941c-03fd363e3bea"
+					(reference "#PWR0107")
+					(unit 1)
+				)
+			)
+		)
+	)
+	(symbol
 		(lib_id "Device:C_Small")
 		(at 179.07 151.13 90)
@@
 					(unit 1)
 				)
+			)
+		)
+	)
+	(symbol
+		(lib_id "Connector_Generic:Conn_01x03")
+		(at 232.41 77.47 0)
+		(unit 1)
+		(body_style 1)
+		(exclude_from_sim no)
+		(in_bom yes)
+		(on_board yes)
+		(in_pos_files yes)
+		(dnp no)
+		(fields_autoplaced yes)
+		(property "Reference" "J101"
+			(at 234.95 76.1999 0)
+			(show_name no)
+			(do_not_autoplace no)
+			(effects
+				(font
+					(size 1.27 1.27)
+				)
+				(justify left)
+			)
+		)
+		(property "Value" "Conn_01x03"
+			(at 234.95 78.7399 0)
+			(show_name no)
+			(do_not_autoplace no)
+			(effects
+				(font
+					(size 1.27 1.27)
+				)
+				(justify left)
+			)
+		)
+		(property "Footprint" "Connector_JST:JST_SH_BM03B-SRSS-TB_1x03-1MP_P1.00mm_Vertical"
+			(at 232.41 77.47 0)
+			(hide yes)
+			(show_name no)
+			(do_not_autoplace no)
+			(effects
+				(font
+					(size 1.27 1.27)
+				)
+			)
+		)
+		(property "Datasheet" ""
+			(at 232.41 77.47 0)
+			(hide yes)
+			(show_name no)
+			(do_not_autoplace no)
+			(effects
+				(font
+					(size 1.27 1.27)
+				)
+			)
+		)
+		(property "Description" "Generic connector, single row, 01x03, script generated (kicad-library-utils/schlib/autogen/connector/)"
+			(at 232.41 77.47 0)
+			(hide yes)
+			(show_name no)
+			(do_not_autoplace no)
+			(effects
+				(font
+					(size 1.27 1.27)
+				)
+			)
+		)
+		(pin "3"
+		)
+		(pin "1"
+		)
+		(pin "2"
+		)
+		(instances
+			(project "pygameboy"
+				(path "/63efa618-1458-4f61-941c-03fd363e3bea"
+					(reference "J101")
+					(unit 1)
+				)

Commit message: WIP v9
Parts:
- removed J1: Conn_01x01, gameboy:Small Hole, symbol Connector_Generic:Conn_01x01
- removed J2: Conn_01x01, gameboy:Large Hole, symbol Connector_Generic:Conn_01x01
- added C103, C104, C105, C106: 10uF, Capacitor_SMD:C_0805_2012Metric, symbol Device:C_Small
- added C107: 100n, Capacitor_SMD:C_0402_1005Metric, symbol Device:C_Small
- added D101: WS2812B-2020, LED_SMD:LED_WS2812B-2020_PLCC4_2.0x2.0mm, symbol LED:WS2812B-2020
- added J102: Conn_01x03, Connector_JST:JST_SH_BM03B-SRSS-TB_1x03-1MP_P1.00mm_Vertical, symbol Connector_Generic:Conn_01x03
- added RN101, RN102, RN103, RN104, RN105, RN106, RN107: 4x1k, Resistor_SMD:R_Array_Convex_4x0603, symbol Device:R_Pack04
- C10, C13: footprint Capacitor_SMD:C_0402_1005Metric -> Capacitor_SMD:C_0603_1608Metric
- D1, D2: value MBR120 -> MBR0540
- U7: value AP2204K-3.3 -> AP2212-3.3
Connections:
- net +3V3: now also C105.2, C106.2, C107.1, D101.4 (VDD); no longer D3.2 (A)
- net +5V: now also C103.2, C104.2
- net A0: now also RN102.4 (R4.1); no longer U1.6 (A0)
- net A1: now also RN102.3 (R3.1); no longer U1.7 (A1)
- net A10: now also RN104.2 (R2.1); no longer U1.16 (A10)
- net A11: now also RN104.1 (R1.1); no longer U1.17 (A11)
- net A12: now also RN105.4 (R4.1); no longer U1.18 (A12)
- net A13: now also RN105.3 (R3.1); no longer U1.19 (A13)
- net A14: now also RN105.2 (R2.1); no longer U1.20 (A14)
- net A15: now also RN105.1 (R1.1); no longer U1.21 (A15)
- net A2: now also RN102.2 (R2.1); no longer U1.8 (A2)
- net A3: now also RN102.1 (R1.1); no longer U1.9 (A3)
- net A4: now also RN103.4 (R4.1); no longer U1.10 (A4)
- net A5: now also RN103.3 (R3.1); no longer U1.11 (A5)
- net A6: now also RN103.2 (R2.1); no longer U1.12 (A6)
- net A7: now also RN103.1 (R1.1); no longer U1.13 (A7)
- net A8: now also RN104.4 (R4.1); no longer U1.14 (A8)
- net A9: now also RN104.3 (R3.1); no longer U1.15 (A9)
- net CLK: now also RN101.4 (R4.1); no longer U1.2 (CLK)
- net CS: now also RN101.1 (R1.1); no longer U1.5 (CS)
- net D0: now also RN106.4 (R4.1); no longer U1.22 (D0)
- net D1: now also RN106.3 (R3.1); no longer U1.23 (D1)
- net D2: now also RN106.2 (R2.1); no longer U1.24 (D2)
- net D3: now also RN106.1 (R1.1); no longer U1.25 (D3)
- net D4: now also RN107.4 (R4.1); no longer U1.26 (D4)
- net D5: now also RN107.3 (R3.1); no longer U1.27 (D5)
- net D6: now also RN107.2 (R2.1); no longer U1.28 (D6)
- net D7: now also RN107.1 (R1.1); no longer U1.29 (D7)
- net GND: now also R4.2, C103.1, C104.1, C105.1, C106.1, C107.2, D101.2 (VSS), J102.2 (Pin_2)
- net LED: now also D3.2 (A); no longer R4.2
- net RD: now also RN101.2 (R2.1); no longer U1.4 (RD)
- net WR: now also RN101.3 (R3.1); no longer U1.3 (WR)
- net +BATT renamed VCC
- new net: RN103.5 (R4.2), U1.10 (A4)
- new net: RN103.6 (R3.2), U1.11 (A5)
- new net: RN103.7 (R2.2), U1.12 (A6)
- new net: RN103.8 (R1.2), U1.13 (A7)
- new net: RN104.5 (R4.2), U1.14 (A8)
- new net: RN104.6 (R3.2), U1.15 (A9)
- new net: RN104.7 (R2.2), U1.16 (A10)
- new net: RN104.8 (R1.2), U1.17 (A11)
- new net: RN105.5 (R4.2), U1.18 (A12)
- new net: RN105.6 (R3.2), U1.19 (A13)
- new net: RN101.5 (R4.2), U1.2 (CLK)
- new net: RN105.7 (R2.2), U1.20 (A14)
- new net: RN105.8 (R1.2), U1.21 (A15)
- new net: RN106.5 (R4.2), U1.22 (D0)
- new net: RN106.6 (R3.2), U1.23 (D1)
- new net: RN106.7 (R2.2), U1.24 (D2)
- new net: RN106.8 (R1.2), U1.25 (D3)
- new net: RN107.5 (R4.2), U1.26 (D4)
- new net: RN107.6 (R3.2), U1.27 (D5)
- new net: RN107.7 (R2.2), U1.28 (D6)
- new net: RN107.8 (R1.2), U1.29 (D7)
- new net: RN101.6 (R3.2), U1.3 (WR)
- new net: RN101.7 (R2.2), U1.4 (RD)
- new net: RN101.8 (R1.2), U1.5 (CS)
- new net: RN102.5 (R4.2), U1.6 (A0)
- new net: RN102.6 (R3.2), U1.7 (A1)
- new net: RN102.7 (R2.2), U1.8 (A2)
- new net: RN102.8 (R1.2), U1.9 (A3)
- new net NEOPIXEL: D101.3 (DIN)
- new net SWCLK: J102.1 (Pin_1)
- new net SWD: J102.3 (Pin_3)
- no-connect marks 4 -> 3
Other:
- sheet RP2350 Core ports: added SWCLK, SWD; removed none
- note added: "GameBoy reset has a pull."
- note added: "TODO: Give space around everything."
- note added: "TODO: Maybe need opamp buffer for sound."
- moved on the sheet: C10, C101, C102, C13, C17, C7, C8, D1, D2, D3, D4, J14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

Commit message: Half routed. microsd added
Parts:
- removed TP1, TP10, TP11, TP12, TP13, TP14, TP15, TP16, TP17, TP18, TP19, TP2, TP20, TP21, TP22, TP23, TP24, TP25, TP26, TP27, TP28, TP29, TP3, TP30, TP31, TP32, TP4, TP5, TP6, TP7, TP8, TP9: Test_Point, gameboy:Test Point, symbol Connector:TestPoint
- added J103: Micro_SD_Card, Adafruit:TF-027-HXXX, symbol Connector:Micro_SD_Card
- added R105: 10k, Resistor_SMD:R_0402_1005Metric, symbol Device:R_Small
- D4: footprint Diode_SMD:D_SOD-123 -> Diode_SMD:D_SOD-523
- J14: footprint Connector_JST:JST_SH_SM04B-SRSS-TB_1x04-1MP_P1.00mm_Horizontal -> Connector_JST:JST_SH_BM04B-SRSS-TB_1x04-1MP_P1.00mm_Vertical
- R6, R7: footprint Resistor_SMD:R_0603_1608Metric -> Resistor_SMD:R_0402_1005Metric
- SW1, SW2: footprint Button_Switch_SMD:SW_SPST_TS-1088-xR020 -> Adafruit:TS-1185
Connections:
- net +3V3: now also J103.4 (VDD), R105.1
- net GND: now also J6.R2, J103.6 (VSS), J103.SH (SHIELD)
- net SHIELD: now also J5.R2
- net at D4.2 (A), J5.R1, U8.2: no longer J5.R2
- net at J6.R1, R7.2: no longer J6.R2
- new net SD_CLK: J103.5 (CLK)
- new net SD_CMD_MOSI: J103.3 (CMD)
- new net SD_DAT0_MISO: J103.7 (DAT0)
- new net SD_DAT1: J103.8 (DAT1)
- new net SD_DAT2: J103.1 (DAT2)
- new net SD_DAT3_CS: J103.2 (DAT3/CD), R105.2
Other:
- sheet RP2350 Core ports: added none; removed GPIO0
- note added: "R2 is S on TRS cables!"
- note added: "SPI0CS"
- note added: "SPI0RX"
- note added: "SPI0SCK"
- note added: "SPI0TX"
- moved on the sheet: C107, D101, D3, R4, R7

Commit message: Final draft of v9
Parts:
- J101, J102: symbol Connector_Generic:Conn_01x03 -> Connector_Generic_MountingPin:Conn_01x03_MountingPin
- J14: symbol Connector_Generic:Conn_01x04 -> Connector_Generic_MountingPin:Conn_01x04_MountingPin
Connections:
- net GND: now also J101.MP (MountPin), J102.MP (MountPin), J14.MP (MountPin)
